File: pcb/recorder/recorder.kicad_pcb (KiCad board)
At the start: 4 copper layers, 605 x 20 mm, 41 parts, among them J1 GPIO_Conn_02x20_Odd_Even, U1 IM73D122V01, U10 TPS7A4700RGWT, U2 ADAU7118, U3 IM73D122V01, U4 IM73D122V01, U5 IM73D122V01, U6 IM73D122V01, U7 IM73D122V01, U8 IM73D122V01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

Commit message: shrunk pcb
Routing:
- net /CLK0: track 537.2 -> 0.00 mm
- net /CLK1: track 534.9 -> 0.00 mm
- net /DAT3: track 379.2 -> 0.00 mm, vias 3 -> 0
- net /DAT0: track 373.7 -> 0.00 mm, vias 3 -> 0
- net /DAT1: track 374.9 -> 2.00 mm, vias 4 -> 1
- net /DAT2: track 375.7 -> 7.28 mm, vias 3 -> 1
- net GND: track 63.4 -> 18.8 mm, vias 30 -> 11
- net /DVDD: track 45.4 -> 9.26 mm, vias 9 -> 2
- net Net-(U3-DATA): track 2.86 -> 0.00 mm
- net Net-(U9-DATA): track 2.86 -> 0.00 mm
- net Net-(U6-DATA): track 2.86 -> 0.00 mm
- net Net-(U4-DATA): track 2.86 -> 0.00 mm
- net Net-(U7-DATA): track 2.86 -> 0.00 mm
- net Net-(U5-DATA): track 3.81 -> 0.95 mm
- net Net-(U1-DATA): track 2.86 -> 0.00 mm
Other:
- board size 605 x 20 mm -> 570 x 20 mm

Commit message: clock traces redone
Parts:
- moved R13 5.36 mm to (428.0, 306.2), turned to -90 degrees
- moved R12 4.74 mm to (424.5, 306.2), turned to -90 degrees
Routing:
- net /CLK1: track 0.00 -> 418.4 mm
- net /CLK0: track 0.00 -> 343.5 mm
- net GND: track 18.8 -> 71.6 mm, vias 11 -> 31
- net /DVDD: track 9.26 -> 39.1 mm, vias 2 -> 6
- net /DAT0: track 0.00 -> 7.16 mm, vias 0 -> 3
- net Net-(U2-PDM_CLK1): track 7.96 -> 2.14 mm
- net /DAT1: track 2.00 -> 7.23 mm, vias 1 -> 3
- net /DAT2: track 7.28 -> 2.22 mm, vias 1 -> 2
- net Net-(U2-PDM_CLK0): track 6.80 -> 2.07 mm
- net Net-(U3-DATA): track 0.00 -> 2.86 mm
- net Net-(U9-DATA): track 0.00 -> 2.86 mm
- net Net-(U6-DATA): track 0.00 -> 2.86 mm
- net Net-(U4-DATA): track 0.00 -> 2.86 mm
- net Net-(U8-DATA): track 0.00 -> 2.86 mm
- net Net-(U7-DATA): track 0.00 -> 2.86 mm
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
Commit message: traces redone, DATA and CLK matched
Routing:
- net /DAT3: track 2.22 -> 362.4 mm, vias 2 -> 3
- net /DAT2: track 2.22 -> 351.6 mm, vias 2 -> 3
- net /DAT0: track 7.16 -> 339.4 mm
- net /DAT1: track 7.23 -> 338.5 mm
- net /DVDD: track 39.1 -> 47.1 mm, vias 6 -> 14
- net /SCLK: track 47.2 -> 46.6 mm

Commit message: DRC updates
Routing:
- net /IOVDD: track 78.8 -> 84.2 mm, vias 1 -> 2
- net /ENABLE: track 7.25 -> 7.90 mm
- net GND: track 71.6 -> 72.0 mm, vias 31 -> 30

Commit message: shrunk to 569 mm
Parts:
- added REF**: MountingHole_4.3mm_M4_ISO14580, Library:MountingHole_4.3mm_M4_ISO14580, F.Cu at (349.0, 300.5)
- added REF**: MountingHole_4.3mm_M4_ISO14580, Library:MountingHole_4.3mm_M4_ISO14580, F.Cu at (549.0, 300.5)
Routing:
- net GND: track 72.0 -> 70.6 mm
Other:
- board size 570 x 20 mm -> 569 x 20 mm
